File: led_cube_cad/led_cube_cad.sch (KiCad schematic (older format))
At the start: 16 parts

Commit message: cad
Parts:
- added B1Q0, B1Q1, B1Q2, B1Q3, B1Q4, B2Q0, B2Q1, B2Q2, B2Q3, B2Q4, B3Q0, B3Q1, B3Q2, B3Q3, B3Q4, B4Q0, B4Q1, B4Q2, B4Q3, B4Q4: BC636, Package_TO_SOT_THT:TO-92_Inline, symbol Transistor_BJT:BC636
- added BoardControl: Conn_01x20, Connector_PinHeader_2.54mm:PinHeader_1x17_P2.54mm_Vertical, symbol Connector_Generic:Conn_01x20
- added CubeConnector: Conn_02x20_Counter_Clockwise, Connector_PinHeader_2.54mm:PinHeader_2x20_P2.54mm_Vertical, symbol Connector_Generic:Conn_02x20_Counter_Clockwise
- added NPN1, NPN2, NPN3, NPN4, NPN5: BC107, Package_TO_SOT_THT:TO-18-3, symbol Transistor_BJT:BC107
- added R? (x20): 10k, symbol Device:R
- added R? (x20): ~100R, symbol Device:R
- added U? (x4): 4099, symbol 4xxx_IEEE:4099
- gave numbers to parts that had none: 5
Connections:
- net Vdd is gone; now on net +5V: U?.16 (Vdd)
- net +5V: now also B1Q0.1 (E), B1Q1.1 (E), B1Q2.1 (E), B1Q3.1 (E), B1Q4.1 (E), B2Q0.1 (E), B2Q1.1 (E), B2Q2.1 (E), B2Q3.1 (E), B2Q4.1 (E), B3Q0.1 (E), B3Q1.1 (E), B3Q2.1 (E), B3Q3.1 (E), B3Q4.1 (E), B4Q0.1 (E), B4Q1.1 (E), B4Q2.1 (E), B4Q3.1 (E), B4Q4.1 (E), BoardControl.1 (Pin_1), U?.16 (Vdd), U?.16 (Vdd), U?.16 (Vdd), U?.16 (Vdd)
- net at U?.2 (R): now also BoardControl.7 (Pin_7), U?.2 (R), U?.2 (R), U?.2 (R), U?.2 (R)
- net at U?.3 (D): now also BoardControl.6 (Pin_6), U?.3 (D), U?.3 (D), U?.3 (D), U?.3 (D)
- net at U?.4 (WR): now also BoardControl.8 (Pin_8)
- net at U?.5 (A0): now also BoardControl.3 (Pin_3), U?.5 (A0), U?.5 (A0), U?.5 (A0), U?.5 (A0)
- net at U?.6 (A1): now also BoardControl.4 (Pin_4), U?.6 (A1), U?.6 (A1), U?.6 (A1), U?.6 (A1)
- net at U?.7 (A2): now also BoardControl.5 (Pin_5), U?.7 (A2), U?.7 (A2), U?.7 (A2), U?.7 (A2)
- net Earth: now reaches U?.8 (Vss)
- net Earth: now also BoardControl.2 (Pin_2), NPN1.1 (E), NPN2.1 (E), NPN3.1 (E), NPN4.1 (E), NPN5.1 (E), U?.8 (Vss), U?.8 (Vss), U?.8 (Vss), U?.8 (Vss)
- net at R?.1: now also CubeConnector.1 (Pin_1)
- net at R?.1: now also CubeConnector.2 (Pin_2)
- net at R?.1: now also CubeConnector.3 (Pin_3)
- net at R?.1: now also CubeConnector.4 (Pin_4)
- net at R?.1: now also CubeConnector.5 (Pin_5)
- new net: B1Q0.2 (C), R?.2
- new net: B1Q0.3 (B), R?.2
- new net: R?.1, U?.10 (Q1) (x4)
- new net: B1Q1.3 (B), R?.2
- new net: R?.1, U?.11 (Q2) (x4)
- new net: B1Q2.3 (B), R?.2
- new net: R?.1, U?.12 (Q3) (x4)
- new net: B1Q3.3 (B), R?.2
- new net: R?.1, U?.13 (Q4) (x4)
- new net: B1Q4.3 (B), R?.2
- new net: R?.1, U?.9 (Q0) (x4)
- new net: BoardControl.9 (Pin_9), U?.4 (WR)
- new net: B1Q1.2 (C), R?.2
- new net: B1Q2.2 (C), R?.2
- new net: B1Q3.2 (C), R?.2
- new net: B1Q4.2 (C), R?.2
- new net: CubeConnector.6 (Pin_6), R?.1
- new net: CubeConnector.7 (Pin_7), R?.1
- new net: CubeConnector.8 (Pin_8), R?.1
- new net: CubeConnector.9 (Pin_9), R?.1
- new net: CubeConnector.10 (Pin_10), R?.1
- new net: B2Q0.2 (C), R?.2
- new net: B2Q0.3 (B), R?.2
- new net: B2Q1.3 (B), R?.2
- new net: B2Q2.3 (B), R?.2
- new net: B2Q3.3 (B), R?.2
- new net: B2Q4.3 (B), R?.2
- new net: BoardControl.10 (Pin_10), U?.4 (WR)
- new net: B2Q1.2 (C), R?.2
- new net: B2Q2.2 (C), R?.2
- new net: B2Q3.2 (C), R?.2
- new net: B2Q4.2 (C), R?.2
- new net: CubeConnector.11 (Pin_11), R?.1
- new net: CubeConnector.12 (Pin_12), R?.1
- new net: CubeConnector.13 (Pin_13), R?.1
- new net: CubeConnector.14 (Pin_14), R?.1
- new net: CubeConnector.15 (Pin_15), R?.1
- new net: B3Q0.2 (C), R?.2
- new net: B3Q0.3 (B), R?.2
- new net: B3Q1.3 (B), R?.2
- new net: B3Q2.3 (B), R?.2
- new net: B3Q3.3 (B), R?.2
- new net: B3Q4.3 (B), R?.2
- new net: BoardControl.11 (Pin_11), U?.4 (WR)
- new net: B3Q1.2 (C), R?.2
- new net: B3Q2.2 (C), R?.2
- new net: B3Q3.2 (C), R?.2
- new net: B3Q4.2 (C), R?.2
- new net: CubeConnector.16 (Pin_16), R?.1
- new net: CubeConnector.17 (Pin_17), R?.1
- new net: CubeConnector.18 (Pin_18), R?.1
- new net: CubeConnector.19 (Pin_19), R?.1
- new net: CubeConnector.20 (Pin_20), R?.1
- new net: B4Q0.2 (C), R?.2
- new net: B4Q0.3 (B), R?.2
- new net: B4Q1.3 (B), R?.2
- new net: B4Q2.3 (B), R?.2
- new net: B4Q3.3 (B), R?.2
- new net: B4Q4.3 (B), R?.2
- new net: BoardControl.12 (Pin_12), U?.4 (WR)
- new net: B4Q1.2 (C), R?.2
- new net: B4Q2.2 (C), R?.2
- new net: B4Q3.2 (C), R?.2
- new net: B4Q4.2 (C), R?.2
- new net: CubeConnector.21 (Pin_21), R?.1
- new net: CubeConnector.22 (Pin_22), R?.1
- new net: CubeConnector.23 (Pin_23), R?.1
- new net: CubeConnector.24 (Pin_24), R?.1
- new net: CubeConnector.25 (Pin_25), R?.1
- new net: CubeConnector.36 (Pin_36), NPN5.3 (C)
- new net: CubeConnector.37 (Pin_37), NPN4.3 (C)
- new net: CubeConnector.38 (Pin_38), NPN3.3 (C)
- new net: CubeConnector.39 (Pin_39), NPN2.3 (C)
- new net: CubeConnector.40 (Pin_40), NPN1.3 (C)
- new net: BoardControl.17 (Pin_17), NPN5.2 (B)
- new net: BoardControl.16 (Pin_16), NPN4.2 (B)
- new net: BoardControl.15 (Pin_15), NPN3.2 (B)
- new net: BoardControl.14 (Pin_14), NPN2.2 (B)
- new net: BoardControl.13 (Pin_13), NPN1.2 (B)
Other:
- moved on the sheet: B0Q0, B0Q1, B0Q2, B0Q3, B0Q4, U?

Commit message: schema
Parts:
- R1, R10, R11, R12, R13, R14, R15, R16, R17, R18, R19, R2, R20, R21, R22, R23, R24, R25, R26, R27, R28, R29, R3, R30, R31, R32, R33, R34, R35, R36, R37, R38, R39, R4, R40, R41, R42, R43, R44, R45, R46, R47, R48, R49, R5, R50, R6, R7, R8, R9: renamed from R?; footprint (none) -> Resistor_THT:R_Axial_DIN0309_L9.0mm_D3.2mm_P12.70mm_Horizontal
- U1, U2, U3, U4, U5: renamed from U?; footprint (none) -> Package_DIP:DIP-16_W10.16mm
- renumbered BoardControl to BoardControl1, CubeConnector to CubeConnector1
Connections:
- no-connect marks 0 -> 23

Commit message: pcb progress
Connections:
- net at R26.1: now also CubeConnector1.9 (Pin_9); no longer CubeConnector1.1 (Pin_1)
- net at R27.1: now also CubeConnector1.7 (Pin_7); no longer CubeConnector1.2 (Pin_2)
- net at R28.1: now also CubeConnector1.5 (Pin_5); no longer CubeConnector1.3 (Pin_3)
- net at R29.1: now also CubeConnector1.3 (Pin_3); no longer CubeConnector1.4 (Pin_4)
- net at R30.1: now also CubeConnector1.1 (Pin_1); no longer CubeConnector1.5 (Pin_5)
- net at R31.1: now also CubeConnector1.19 (Pin_19); no longer CubeConnector1.6 (Pin_6)
- net at R32.1: now also CubeConnector1.17 (Pin_17); no longer CubeConnector1.7 (Pin_7)
- net at R33.1: now also CubeConnector1.15 (Pin_15); no longer CubeConnector1.8 (Pin_8)
- net at R34.1: now also CubeConnector1.13 (Pin_13); no longer CubeConnector1.9 (Pin_9)
- net at R35.1: now also CubeConnector1.11 (Pin_11); no longer CubeConnector1.10 (Pin_10)
- net at R36.1: now also CubeConnector1.29 (Pin_29); no longer CubeConnector1.11 (Pin_11)
- net at R37.1: now also CubeConnector1.27 (Pin_27); no longer CubeConnector1.12 (Pin_12)
- net at R38.1: now also CubeConnector1.25 (Pin_25); no longer CubeConnector1.13 (Pin_13)
- net at R39.1: now also CubeConnector1.23 (Pin_23); no longer CubeConnector1.14 (Pin_14)
- net at R40.1: now also CubeConnector1.21 (Pin_21); no longer CubeConnector1.15 (Pin_15)
- net at R41.1: now also CubeConnector1.39 (Pin_39); no longer CubeConnector1.16 (Pin_16)
- net at R42.1: now also CubeConnector1.37 (Pin_37); no longer CubeConnector1.17 (Pin_17)
- net at R43.1: now also CubeConnector1.35 (Pin_35); no longer CubeConnector1.18 (Pin_18)
- net at R44.1: now also CubeConnector1.33 (Pin_33); no longer CubeConnector1.19 (Pin_19)
- net at R45.1: now also CubeConnector1.31 (Pin_31); no longer CubeConnector1.20 (Pin_20)
- net at R46.1: now also CubeConnector1.40 (Pin_40); no longer CubeConnector1.21 (Pin_21)
- net at R47.1: now also CubeConnector1.38 (Pin_38); no longer CubeConnector1.22 (Pin_22)
- net at R48.1: now also CubeConnector1.36 (Pin_36); no longer CubeConnector1.23 (Pin_23)
- net at R49.1: now also CubeConnector1.34 (Pin_34); no longer CubeConnector1.24 (Pin_24)
- net at R50.1: now also CubeConnector1.32 (Pin_32); no longer CubeConnector1.25 (Pin_25)
- net at NPN5.3 (C): no longer CubeConnector1.36 (Pin_36)
- net at NPN4.3 (C): no longer CubeConnector1.37 (Pin_37)
- net at NPN3.3 (C): no longer CubeConnector1.38 (Pin_38)
- net at NPN2.3 (C): no longer CubeConnector1.39 (Pin_39)
- net at NPN1.3 (C): no longer CubeConnector1.40 (Pin_40)
- net at NPN5.2 (B): no longer BoardControl1.17 (Pin_17)
- net at NPN4.2 (B): no longer BoardControl1.16 (Pin_16)
- net at NPN3.2 (B): no longer BoardControl1.15 (Pin_15)
- net at NPN2.2 (B): no longer BoardControl1.14 (Pin_14)
- net at NPN1.2 (B): no longer BoardControl1.13 (Pin_13)
- net Earth renamed GND
- no-connect marks 23 -> 13
Other:
- moved on the sheet: NPN1, NPN2, NPN3, NPN4, NPN5

Commit message: some routes
Parts:
- added RL0, RL1, RL2, RL3, RL4: 10k, Resistor_THT:R_Axial_DIN0309_L9.0mm_D3.2mm_P12.70mm_Horizontal, symbol Device:R
- B0Q0: value BC636 -> BC560; footprint Package_TO_SOT_THT:TO-92_Inline -> Package_TO_SOT_THT:TO-92; symbol Transistor_BJT:BC636 -> Transistor_BJT:BC560
- B0Q1, B0Q2, B0Q3, B0Q4, B1Q0, B1Q1, B1Q2, B1Q3, B1Q4, B2Q0, B2Q1, B2Q2, B2Q3, B2Q4, B3Q0, B3Q1, B3Q2, B3Q3, B3Q4, B4Q0, B4Q1, B4Q2, B4Q3, B4Q4: value BC636 -> BC560; symbol Transistor_BJT:BC636 -> Transistor_BJT:BC560
Connections:
- net +5V: now also B0Q0.3 (E), B0Q1.3 (E), B0Q2.3 (E), B0Q3.3 (E), B0Q4.3 (E), B1Q0.3 (E), B1Q1.3 (E), B1Q2.3 (E), B1Q3.3 (E), B1Q4.3 (E), B2Q0.3 (E), B2Q1.3 (E), B2Q2.3 (E), B2Q3.3 (E), B2Q4.3 (E), B3Q0.3 (E), B3Q1.3 (E), B3Q2.3 (E), B3Q3.3 (E), B3Q4.3 (E), B4Q0.3 (E), B4Q1.3 (E), B4Q2.3 (E), B4Q3.3 (E), B4Q4.3 (E); no longer B0Q0.1 (E), B0Q1.1 (E), B0Q2.1 (E), B0Q3.1 (E), B0Q4.1 (E), B1Q0.1 (E), B1Q1.1 (E), B1Q2.1 (E), B1Q3.1 (E), B1Q4.1 (E), B2Q0.1 (E), B2Q1.1 (E), B2Q2.1 (E), B2Q3.1 (E), B2Q4.1 (E), B3Q0.1 (E), B3Q1.1 (E), B3Q2.1 (E), B3Q3.1 (E), B3Q4.1 (E), B4Q0.1 (E), B4Q1.1 (E), B4Q2.1 (E), B4Q3.1 (E), B4Q4.1 (E)
- net at R26.2: now also B0Q0.1 (C); no longer B0Q0.2 (C)
- net at R1.2: now also B0Q0.2 (B); no longer B0Q0.3 (B)
- net at R2.2: now also B0Q1.2 (B); no longer B0Q1.3 (B)
- net at R3.2: now also B0Q2.2 (B); no longer B0Q2.3 (B)
- net at R4.2: now also B0Q3.2 (B); no longer B0Q3.3 (B)
- net at R5.2: now also B0Q4.2 (B); no longer B0Q4.3 (B)
- net at R27.2: now also B0Q1.1 (C); no longer B0Q1.2 (C)
- net at R28.2: now also B0Q2.1 (C); no longer B0Q2.2 (C)
- net at R29.2: now also B0Q3.1 (C); no longer B0Q3.2 (C)
- net at R30.2: now also B0Q4.1 (C); no longer B0Q4.2 (C)
- net at R31.2: now also B1Q0.1 (C); no longer B1Q0.2 (C)
- net at R6.2: now also B1Q0.2 (B); no longer B1Q0.3 (B)
- net at R7.2: now also B1Q1.2 (B); no longer B1Q1.3 (B)
- net at R8.2: now also B1Q2.2 (B); no longer B1Q2.3 (B)
- net at R9.2: now also B1Q3.2 (B); no longer B1Q3.3 (B)
- net at R10.2: now also B1Q4.2 (B); no longer B1Q4.3 (B)
- net at R32.2: now also B1Q1.1 (C); no longer B1Q1.2 (C)
- net at R33.2: now also B1Q2.1 (C); no longer B1Q2.2 (C)
- net at R34.2: now also B1Q3.1 (C); no longer B1Q3.2 (C)
- net at R35.2: now also B1Q4.1 (C); no longer B1Q4.2 (C)
- net at R36.2: now also B2Q0.1 (C); no longer B2Q0.2 (C)
- net at R11.2: now also B2Q0.2 (B); no longer B2Q0.3 (B)
- net at R12.2: now also B2Q1.2 (B); no longer B2Q1.3 (B)
- net at R13.2: now also B2Q2.2 (B); no longer B2Q2.3 (B)
- net at R14.2: now also B2Q3.2 (B); no longer B2Q3.3 (B)
- net at R15.2: now also B2Q4.2 (B); no longer B2Q4.3 (B)
- net at R37.2: now also B2Q1.1 (C); no longer B2Q1.2 (C)
- net at R38.2: now also B2Q2.1 (C); no longer B2Q2.2 (C)
- net at R39.2: now also B2Q3.1 (C); no longer B2Q3.2 (C)
- net at R40.2: now also B2Q4.1 (C); no longer B2Q4.2 (C)
- net at R41.2: now also B3Q0.1 (C); no longer B3Q0.2 (C)
- net at R16.2: now also B3Q0.2 (B); no longer B3Q0.3 (B)
- net at R17.2: now also B3Q1.2 (B); no longer B3Q1.3 (B)
- net at R18.2: now also B3Q2.2 (B); no longer B3Q2.3 (B)
- net at R19.2: now also B3Q3.2 (B); no longer B3Q3.3 (B)
- net at R20.2: now also B3Q4.2 (B); no longer B3Q4.3 (B)
- net at R42.2: now also B3Q1.1 (C); no longer B3Q1.2 (C)
- net at R43.2: now also B3Q2.1 (C); no longer B3Q2.2 (C)
- net at R44.2: now also B3Q3.1 (C); no longer B3Q3.2 (C)
- net at R45.2: now also B3Q4.1 (C); no longer B3Q4.2 (C)
- net at R46.2: now also B4Q0.1 (C); no longer B4Q0.2 (C)
- net at R21.2: now also B4Q0.2 (B); no longer B4Q0.3 (B)
- net at R22.2: now also B4Q1.2 (B); no longer B4Q1.3 (B)
- net at R23.2: now also B4Q2.2 (B); no longer B4Q2.3 (B)
- net at R24.2: now also B4Q3.2 (B); no longer B4Q3.3 (B)
- net at R25.2: now also B4Q4.2 (B); no longer B4Q4.3 (B)
- net at R47.2: now also B4Q1.1 (C); no longer B4Q1.2 (C)
- net at R48.2: now also B4Q2.1 (C); no longer B4Q2.2 (C)
- net at R49.2: now also B4Q3.1 (C); no longer B4Q3.2 (C)
- net at R50.2: now also B4Q4.1 (C); no longer B4Q4.2 (C)
- net at CubeConnector1.22 (Pin_22): now also NPN1.3 (C)
- net at CubeConnector1.24 (Pin_24): now also NPN2.3 (C)
- net at CubeConnector1.26 (Pin_26): now also NPN3.3 (C)
- net at CubeConnector1.28 (Pin_28): now also NPN4.3 (C)
- net at CubeConnector1.30 (Pin_30): now also NPN5.3 (C)
- net at NPN5.2 (B): now also RL4.2
- net at NPN4.2 (B): now also RL3.2
- net at NPN3.2 (B): now also RL2.2
- net at NPN2.2 (B): now also RL1.2
- net at NPN1.2 (B): now also RL0.2
- net at BoardControl1.13 (Pin_13): now also RL0.1
- net at BoardControl1.14 (Pin_14): now also RL1.1
- net at BoardControl1.15 (Pin_15): now also RL2.1
- net at BoardControl1.16 (Pin_16): now also RL3.1
- net at BoardControl1.17 (Pin_17): now also RL4.1
Other:
- moved on the sheet: NPN1, NPN2, NPN3, NPN4, NPN5

Commit message: backup
Connections:
- net at R46.1: now also CubeConnector1.32 (Pin_32); no longer CubeConnector1.40 (Pin_40)
- net at R47.1: now also CubeConnector1.34 (Pin_34); no longer CubeConnector1.38 (Pin_38)
- net at R49.1: now also CubeConnector1.38 (Pin_38); no longer CubeConnector1.34 (Pin_34)
- net at R50.1: now also CubeConnector1.40 (Pin_40); no longer CubeConnector1.32 (Pin_32)
Changed lines of the file:
@@
 	5950 13350 9300 13350
 Wire Wire Line
-	9300 7400 8750 7400
+	9300 8200 9300 13350
 Wire Wire Line
-	9300 7400 9300 13350
-Wire Wire Line
-	9350 7600 8750 7600
-Wire Wire Line
-	9350 7600 9350 13600
-Wire Wire Line
-	9400 7800 8750 7800
+	9350 8000 9350 13600
 Wire Wire Line
 	9400 7800 9400 13850
 Wire Wire Line
-	9450 8000 8750 8000
+	9450 7600 9450 14100
 Wire Wire Line
-	9450 8000 9450 14100
-Wire Wire Line
-	9500 8200 8750 8200
-Wire Wire Line
-	9500 8200 9500 14350
+	9500 7400 9500 14350
 Wire Wire Line
 	8750 9200 10100 9200
@@
 Wire Wire Line
 	11150 7450 11150 12650
+Wire Wire Line
+	9500 7400 8750 7400
+Wire Wire Line
+	8750 7600 9450 7600
+Wire Wire Line
+	8750 7800 9400 7800
+Wire Wire Line
+	8750 8000 9350 8000
+Wire Wire Line
+	8750 8200 9300 8200
 $EndSCHEMATC

Commit message: addressing wired
Connections:
- net at U1.5 (A0), U2.5 (A0), U3.5 (A0)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: now also BoardControl1.5 (Pin_5); no longer BoardControl1.3 (Pin_3)
- net at U1.7 (A2), U2.7 (A2), U3.7 (A2)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: now also BoardControl1.3 (Pin_3); no longer BoardControl1.5 (Pin_5)
Changed lines of the file:
@@
 Wire Wire Line
 	1200 12900 1200 13950
-Wire Wire Line
-	1200 13950 1250 13950
-Wire Wire Line
-	1250 13950 1250 14350
 Connection ~ 1200 12900
 Wire Wire Line
-	1100 12800 1100 14000
-Wire Wire Line
-	1100 14000 1150 14000
-Wire Wire Line
-	1150 14000 1150 14350
-Connection ~ 1100 12800
-Wire Wire Line
 	1000 12700 1000 14050
-Wire Wire Line
-	1000 14050 1050 14050
-Wire Wire Line
-	1050 14050 1050 14350
 Connection ~ 1000 12700
 Wire Wire Line
@@
 Wire Wire Line
 	8750 8200 9300 8200
+Wire Wire Line
+	1250 14050 1250 14350
+Wire Wire Line
+	1000 14050 1250 14050
+Wire Wire Line
+	1150 13450 1150 14350
+Wire Wire Line
+	1050 13950 1050 14350
+Wire Wire Line
+	1050 13950 1200 13950
+Wire Wire Line
+	1100 12800 1100 13450
+Wire Wire Line
+	1100 13450 1150 13450
+Connection ~ 1100 12800
 $EndSCHEMATC

Commit message: pads
Parts:
- added DATA1, DATA2, DATA3, DATA4, DATA5, RESET1, RESET2, RESET3, RESET4, RESET5: Conn_01x01_Female, TestPoint:TestPoint_THTPad_D1.5mm_Drill0.7mm, symbol Connector:Conn_01x01_Female
Connections:
- net at BoardControl1.7 (Pin_7), U1.2 (R), U2.2 (R)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: now also RESET1.1 (Pin_1), RESET2.1 (Pin_1), RESET3.1 (Pin_1), RESET4.1 (Pin_1), RESET5.1 (Pin_1)
- net at BoardControl1.6 (Pin_6), U1.3 (D), U2.3 (D)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: now also DATA1.1 (Pin_1), DATA2.1 (Pin_1), DATA3.1 (Pin_1), DATA4.1 (Pin_1), DATA5.1 (Pin_1)
Changed lines of the file:
@@
 	1200 12900 2300 12900
 Wire Wire Line
-	2300 13100 1300 13100
-Wire Wire Line
-	1300 1750 2300 1750
-Wire Wire Line
-	2300 4650 1300 4650
+	2300 13100 2050 13100
+Wire Wire Line
+	1300 1750 1800 1750
+Wire Wire Line
+	2300 4650 1900 4650
 Connection ~ 1300 4650
 Wire Wire Line
@@
 	1200 7300 1200 10100
 Wire Wire Line
-	2300 7500 1300 7500
+	2300 7500 1850 7500
 Connection ~ 1300 7500
 Wire Wire Line
@@
 	1200 10100 1200 12900
 Wire Wire Line
-	2300 10300 1300 10300
+	2300 10300 2000 10300
 Connection ~ 1300 10300
 Wire Wire Line
 	1300 10300 1300 7500
 Wire Wire Line
-	2300 1850 1400 1850
-Wire Wire Line
 	1400 1850 1400 4750
 Wire Wire Line
-	1400 13200 2300 13200
-Wire Wire Line
-	2300 10400 1400 10400
+	1400 13200 2150 13200
 Connection ~ 1400 10400
 Wire Wire Line
 	1400 10400 1400 13200
-Wire Wire Line
-	2300 7600 1400 7600
 Connection ~ 1400 7600
 Wire Wire Line
 	1400 7600 1400 10400
 Wire Wire Line
-	2300 4750 1400 4750
+	2300 4750 2000 4750
 Connection ~ 1400 4750
 Wire Wire Line
@@
 	1100 13450 1150 13450
 Connection ~ 1100 12800
+$Comp
+L Connector:Conn_01x01_Female RESET1
+U 1 1 5FD3CE35
+P 2050 2100
+F 0 "RESET1" H 2078 2080 50  0000 L CNN
+F 1 "Conn_01x01_Female" H 2078 2035 50  0001 L CNN
+F 2 "TestPoint:TestPoint_THTPad_D1.5mm_Drill0.7mm" H 2050 2100 50  0001 C CNN
+F 3 "~" H 2050 2100 50  0001 C CNN
+	1    2050 2100
+	1    0    0    -1
+$EndComp
+$Comp
+L Connector:Conn_01x01_Female DATA1
+U 1 1 5FD84EDE
+P 2050 2300
+F 0 "DATA1" H 2078 2280 50  0000 L CNN
+F 1 "Conn_01x01_Female" H 2078 2235 50  0001 L CNN
+F 2 "TestPoint:TestPoint_THTPad_D1.5mm_Drill0.7mm" H 2050 2300 50  0001 C CNN
+F 3 "~" H 2050 2300 50  0001 C CNN
+	1    2050 2300
+	1    0    0    -1
+$EndComp
+Wire Wire Line
+	1850 2100 1850 1850
+Wire Wire Line
+	1400 1850 1850 1850
+Connection ~ 1850 1850
+Wire Wire Line
+	1850 1850 2300 1850
+Wire Wire Line
+	1850 2300 1800 2300
+Wire Wire Line
+	1800 2300 1800 1750
+Connection ~ 1800 1750
+Wire Wire Line
+	1800 1750 2300 1750
+$Comp
+L Connector:Conn_01x01_Female DATA2
+U 1 1 5FE9BF60
+P 2200 5200
+F 0 "DATA2" H 2228 5180 50  0000 L CNN
+F 1 "Conn_01x01_Female" H 2228 5135 50  0001 L CNN
+F 2 "TestPoint:TestPoint_THTPad_D1.5mm_Drill0.7mm" H 2200 5200 50  0001 C CNN
+F 3 "~" H 2200 5200 50  0001 C CNN
+	1    2200 5200
+	1    0    0    -1
+$EndComp
+$Comp
+L Connector:Conn_01x01_Female RESET2
+U 1 1 5FEDD4E6
+P 2200 4950
+F 0 "RESET2" H 2228 4930 50  0000 L CNN
+F 1 "Conn_01x01_Female" H 2228 4885 50  0001 L CNN
+F 2 "TestPoint:TestPoint_THTPad_D1.5mm_Drill0.7mm" H 2200 4950 50  0001 C CNN
+F 3 "~" H 2200 4950 50  0001 C CNN
+	1    2200 4950
+	1    0    0    -1
+$EndComp
+$Comp
+L Connector:Conn_01x01_Female DATA3
+U 1 1 5FF20AB6
+P 2150 8050
+F 0 "DATA3" H 2178 8030 50  0000 L CNN
+F 1 "Conn_01x01_Female" H 2178 7985 50  0001 L CNN
+F 2 "TestPoint:TestPoint_THTPad_D1.5mm_Drill0.7mm" H 2150 8050 50  0001 C CNN
+F 3 "~" H 2150 8050 50  0001 C CNN
+	1    2150 8050
+	1    0    0    -1
+$EndComp
+$Comp
+L Connector:Conn_01x01_Female RESET3
+U 1 1 5FF20ABC
+P 2150 7800
+F 0 "RESET3" H 2178 7780 50  0000 L CNN
+F 1 "Conn_01x01_Female" H 2178 7735 50  0001 L CNN
+F 2 "TestPoint:TestPoint_THTPad_D1.5mm_Drill0.7mm" H 2150 7800 50  0001 C CNN
+F 3 "~" H 2150 7800 50  0001 C CNN
+	1    2150 7800
+	1    0    0    -1
+$EndComp
+$Comp
+L Connector:Conn_01x01_Female DATA4
+U 1 1 5FF623A3
+P 2250 10850
+F 0 "DATA4" H 2278 10830 50  0000 L CNN
+F 1 "Conn_01x01_Female" H 2278 10785 50  0001 L CNN
+F 2 "TestPoint:TestPoint_THTPad_D1.5mm_Drill0.7mm" H 2250 10850 50  0001 C CNN
+F 3 "~" H 2250 10850 50  0001 C CNN
+	1    2250 10850
+	1    0    0    -1
+$EndComp
+$Comp
+L Connector:Conn_01x01_Female RESET4
+U 1 1 5FF623A9
+P 2250 10600
+F 0 "RESET4" H 2278 10580 50  0000 L CNN
+F 1 "Conn_01x01_Female" H 2278 10535 50  0001 L CNN
+F 2 "TestPoint:TestPoint_THTPad_D1.5mm_Drill0.7mm" H 2250 10600 50  0001 C CNN
+F 3 "~" H 2250 10600 50  0001 C CNN
+	1    2250 10600
+	1    0    0    -1
+$EndComp
+$Comp
+L Connector:Conn_01x01_Female DATA5
+U 1 1 5FFA3CC2
+P 2350 13600
+F 0 "DATA5" H 2378 13580 50  0000 L CNN
+F 1 "Conn_01x01_Female" H 2378 13535 50  0001 L CNN
+F 2 "TestPoint:TestPoint_THTPad_D1.5mm_Drill0.7mm" H 2350 13600 50  0001 C CNN
+F 3 "~" H 2350 13600 50  0001 C CNN
+	1    2350 13600
+	1    0    0    -1
+$EndComp
+$Comp
+L Connector:Conn_01x01_Female RESET5
+U 1 1 5FFA3CC8
+P 2350 13350
+F 0 "RESET5" H 2378 13330 50  0000 L CNN
+F 1 "Conn_01x01_Female" H 2378 13285 50  0001 L CNN
+F 2 "TestPoint:TestPoint_THTPad_D1.5mm_Drill0.7mm" H 2350 13350 50  0001 C CNN
+F 3 "~" H 2350 13350 50  0001 C CNN
+	1    2350 13350
+	1    0    0    -1
+$EndComp
+Wire Wire Line
+	2150 13350 2150 13200
+Connection ~ 2150 13200
+Wire Wire Line
+	2150 13200 2300 13200
+Wire Wire Line
+	2050 13100 2050 13600
+Wire Wire Line
+	2050 13600 2150 13600
+Connection ~ 2050 13100
+Wire Wire Line
+	2050 13100 1300 13100
+Wire Wire Line
+	2050 10600 2050 10400
+Wire Wire Line
+	1400 10400 2050 10400
+Connection ~ 2050 10400
+Wire Wire Line
+	2050 10400 2300 10400
+Wire Wire Line
+	2050 10850 2000 10850
+Wire Wire Line
+	2000 10850 2000 10300
+Connection ~ 2000 10300
+Wire Wire Line
+	2000 10300 1300 10300
+Wire Wire Line
+	1950 7800 1950 7600
+Wire Wire Line
+	1400 7600 1950 7600
+Connection ~ 1950 7600
+Wire Wire Line
+	1950 7600 2300 7600
+Wire Wire Line
+	1950 8050 1850 8050
+Wire Wire Line
+	1850 8050 1850 7500
+Connection ~ 1850 7500
+Wire Wire Line
+	1850 7500 1300 7500
+Wire Wire Line
+	2000 4950 2000 4750
+Connection ~ 2000 4750
+Wire Wire Line
+	2000 4750 1400 4750
+Wire Wire Line
+	2000 5200 1900 5200
+Wire Wire Line
+	1900 5200 1900 4650
+Connection ~ 1900 4650
+Wire Wire Line
+	1900 4650 1300 4650
 $EndSCHEMATC
